File: ESP32WithWriter.kicad_sch (KiCad schematic)
At the start: 24 parts, among them J1 USB_C_Receptacle_USB2.0, SW1 SW_Push, SW2 SW_Push, U1 ESP32-WROOM-32D, U2 AMS1117-3.3, U3 CH340K

Commit message: 32D->S3N16
Parts:
- removed C4, C5: 103, Capacitor_SMD:C_0603_1608Metric_Pad1.08x0.95mm_HandSolder, symbol Device:C
- removed R4, R5: 101, Resistor_SMD:R_0603_1608Metric_Pad0.98x0.95mm_HandSolder, symbol Device:R
- removed U3: CH340K, Package_SO:SSOP-10_3.9x4.9mm_P1.00mm, symbol Interface_USB:CH340K
- U1: value ESP32-WROOM-32D -> ESP32-S3-WROOM-1; footprint RF_Module:ESP32-WROOM-32 -> RF_Module:ESP32-S3-WROOM-1; symbol RF_Module:ESP32-WROOM-32D -> RF_Module:ESP32-S3-WROOM-1
Connections:
- net ESP-RXD2: now also U1.8 (IO15); no longer U1.27 (IO16)
- net ESP-TXD2: now also U1.9 (IO16); no longer U1.28 (IO17)
- net ESP_IO0: now also U1.27 (IO0); no longer U1.25 (IO0)
- net GND: now also U1.40 (GND), U1.41 (GND); no longer U1.15 (GND), U1.38 (GND), U1.39 (GND)
- net HSPI-MISO: now also U1.21 (IO13); no longer U1.14 (IO12)
- net HSPI-MOSI: now also U1.22 (IO14); no longer U1.16 (IO13)
- net HSPI-SCK: now also U1.20 (IO12); no longer U1.13 (IO14)
- net I2C0-SCL: now also U1.17 (IO9); no longer U1.36 (IO22)
- net I2C0-SDA: now also U1.12 (IO8); no longer U1.33 (IO21)
- net I2C1-SCL: now also U1.19 (IO11); no longer U1.8 (IO32)
- net I2C1-SDA: now also U1.18 (IO10); no longer U1.9 (IO33)
- net IO2: now also U1.38 (IO2); no longer U1.24 (IO2)
- net IO27: now also U1.33 (IO40); no longer U1.12 (IO27)
- net IO35: now also U1.28 (IO35); no longer U1.7 (IO35)
- net SD-CD: now also U1.32 (IO39); no longer U1.29 (IO5)
- net SD-CLK: now also U1.29 (IO36); no longer U1.30 (IO18)
- net SD-CMD: now also U1.31 (IO38); no longer U1.37 (IO23)
- net SD-D0: now also U1.30 (IO37); no longer U1.31 (IO19)
- net USB-D+: now also U1.14 (USB_D+)
- net USB-D-: now also U1.13 (USB_D-)
- net +3V3 renamed 3V3
- net DTR-H: no longer names the net of R8.2, R9.1
- net ESP-RXD0: no longer names the net of U1.34 (IO41)
- net ESP-TXD0: no longer names the net of U1.35 (IO42)
- net IO34 renamed IO6
- net IO4: no longer names the net of U1.26 (IO45)
- net RTS-H: no longer names the net of R6.2, R7.1
- net SVN_IO39 renamed IO5
- net SVP_IO36: no longer names the net of U1.4 (IO4)
- new net IO1: U1.39 (IO1)
- new net IO7: U1.7 (IO7)
- no-connect marks 10 -> 13
